Commit message: update and use the correted urdf file by enyu but still need to implement PID control for the y_joints constraints

File: assets/robot_raw/stretch_description_RE2V0_fake_joint.urdf (robot description, URDF)
Before this commit: robot stretch, 48 links, 47 joints
Links:
- removed link rotate_link_z
- added link virtual_link_x
- added link virtual_link_y
- added link virtual_link_z
- link link_gripper_fingertip_left: mass 0.003822 -> 0.05
- link link_gripper_fingertip_right: mass 0.003822 -> 0.05
Joints:
- removed joint base_forward
- removed joint rotate_z
- added joint joint_base: type fixed, parent virtual_link_z, child base_link, origin xyz=0 0 0 rpy=0 0 0, axis 0 0 0
- added joint joint_rot_z: type revolute, parent virtual_link_y, child virtual_link_z, origin xyz=0 0 0 rpy=0 0 0, axis 0 0 1, limit lower=-31.4 upper=31.4 effort=100 velocity=1.5
- added joint joint_x: type prismatic, parent base_ground, child virtual_link_x, origin xyz=0 0 0 rpy=0 0 0, axis 1 0 0, limit lower=-10.0 upper=10.0 effort=100 velocity=1.0
- added joint joint_y: type prismatic, parent virtual_link_x, child virtual_link_y, origin xyz=0 0 0 rpy=0 0 0, axis 0 1 0, limit lower=-10.0 upper=10.0 effort=100 velocity=1.0
